File: BE_elec_ampli_audio.kicad_pcb (KiCad board)
At the start: 2 copper layers, 52 parts, among them J2 Conn_01x02, J3 Conn_01x03, Q1 Q_PNP_EBC, Q10 Q_PNP_BCE, Q11 BD139, Q12 Q_PNP_BCE, Q13 Q_NPN_EBC, Q2 Q_PNP_EBC, Q3 Q_PNP_EBC, Q4 Q_NPN_EBC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

Commit message: kicad_pcb
Parts:
- added D3: 1N4001, CmpAmpliAudio:D_DO-35_SOD27_P10.16mm_Horizontal, F.Cu at (119.4, 33.0)
- added D4: 1N4001, CmpAmpliAudio:D_DO-35_SOD27_P10.16mm_Horizontal, F.Cu at (115.6, 26.7)
- moved R1 181.3 mm to (47.0, 104.1), turned to 270 degrees
- moved R11 163.1 mm to (128.3, 110.5), turned to 90 degrees
- moved Q1 159.4 mm to (53.3, 92.7), turned to 270 degrees
- moved C2 149.6 mm to (83.8, 106.7), turned to 180 degrees
- moved RV2 149.1 mm to (81.3, 86.4)
- moved Q5 148.4 mm to (94.0, 99.1), turned to 90 degrees
- moved C1 146.1 mm to (55.9, 105.4)
- moved R2 145.4 mm to (61.0, 95.2)
- moved Q8 142.2 mm to (94.0, 74.9), turned to 180 degrees
- moved C11 140.6 mm to (111.8, 85.1), turned to 180 degrees
- moved R8 139.2 mm to (88.9, 90.2)
- moved Q3 138.6 mm to (40.6, 85.1)
- moved Q4 136.0 mm to (82.5, 96.5), turned to 270 degrees
- moved R12 135.7 mm to (102.9, 109.2)
- moved Q13 127.4 mm to (73.7, 50.8), turned to 90 degrees
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