File: BE_elec_ampli_audio.sch (KiCad schematic (older format))
At the start: 52 parts, among them J2 Conn_01x02, J3 Conn_01x03, Q1 Q_PNP_EBC, Q10 Q_PNP_BCE, Q11 BD139, Q12 Q_PNP_BCE, Q13 Q_NPN_EBC, Q2 Q_PNP_EBC, Q3 Q_PNP_EBC, Q4 Q_NPN_EBC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

Commit message: .sch
Parts:
- added D3, D4: 1N4001, CmpAmpliAudio:D_DO-35_SOD27_P10.16mm_Horizontal, symbol Diode:1N4148
Connections:
- net +12V: now also D3.1 (K)
- net -12V: now also D4.2 (A)
- net GND: now also D3.2 (A), D4.1 (K)
